File: hardware/gecko_power_supply_transmitter/rev_a/gpst_a.brd (EAGLE design)
At the start: 32.5 x 13 mm, 33 parts, among them J2 GECKO_POWER_SUPPLY_CONN, J3 TC2030-CTX-NL, Q2 MOSFET-NCHANNELXFDN-3, U1 DS2411, U2 FM25LBTDFN-8, U4 CC2538, X1 EPSON-FA-128

Commit message: got rf routed
added silkscreen
Parts:
- moved A1 0.25 mm to (3.81, 6.50)
Connections:
- net N$5 renamed RF_P
- net N$6 renamed RF_N
- net N$7 renamed ANTENNA
Routing:
- net GND: track 12.2 -> 16.1 mm, vias 37 -> 42
- net RF_N: track 3.04 -> 0.00 mm
- net RF_P: track 3.03 -> 0.00 mm
- added copper zone on layer 1, net ANTENNA
- added copper zone on layer 1, net RF_N
- added copper zone on layer 1, net RF_P
Other:
- board text added: "2013/08/12"
- board text added: "Brad Campbell"
- board text added: "sEHnsor"

Commit message: bom and new pdfs
Parts:
- removed C17: 1uF, passives:0402_CAP
- removed C18: 2.2uF, passives:0402_CAP
- removed J3: TC2030-CTX-NL, connector:TC2030-IDC-NL
- added C3: 220pF, passives:0402_CAP
- added C4: 1nF, passives:0402_CAP
- added J1: GECKO_POWER_SUPPLY_CONN, gecko:HEADER1X6/0.05IN
- C1: value 0.1uF -> 12pF
- C10, C11, C12, C8, C9: value 100nF -> 0.1uF
- C13: value 220pF -> 1uF
- C14, C15: value 100nF -> 1uF
- C16: value 1uF -> 2.2uF
- C2: value 1nF -> 12pF
- C5, C6: value 12pF -> 0.1uF
- C7: value 1uF -> 0.1uF
- J2: value GECKO_POWER_SUPPLY_CONN -> TC2030-CTX-NL; device gecko:HEADER1X6/0.05IN -> connector:TC2030-IDC-NL
- R1: value 4.7k -> 2.2k
- R5: value 2.2k -> 4.7k
- R6: value 4.7M -> 56k
- R7: value 56k -> 4.7M
- moved R6 16.4 mm to (11.7, 0.85), turned to 180 degrees
- moved R7 16.4 mm to (23.5, 12.2), turned to 0 degrees
- moved C15 13.3 mm to (21.8, 0.82), turned to 0 degrees
- moved R1 12.4 mm to (15.5, 11.7), turned to 270 degrees
- moved C10 12.2 mm to (11.0, 7.78), turned to 180 degrees
- moved C1 12.2 mm to (13.4, 11.7), turned to 90 degrees
- moved C5 12.2 mm to (25.6, 12.0), turned to 0 degrees
- moved R2 11.4 mm to (24.0, 4.14), turned to 180 degrees
- moved C16 10.6 mm to (23.5, 11.3), turned to 180 degrees
- moved C14 9.14 mm to (11.0, 9.43), turned to 180 degrees
- moved C13 7.79 mm to (19.4, 1.02)
- moved C7 7.40 mm to (23.3, 7.33), turned to 0 degrees
- moved R3 6.85 mm to (26.2, 5.40), turned to 180 degrees
- moved R4 6.58 mm to (28.2, 12.0)
- moved J2 6.09 mm to (29.2, 2.05), turned to 180 degrees
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- renumbered Q2 to Q1, U4 to U3
Connections:
- net !FRAM_CS: now also R3.1; no longer R1.1
- net !FRAM_HOLD: now also R4.1; no longer R3.1
- net !FRAM_WP: now also R5.1; no longer R4.1
- net !RESET: now also J2.3, R1.1; no longer J3.3, R2.1
- net DS2411: now also R2.1; no longer R5.1
- net GND: now also C3.2, C4.2, J1.1, J2.5, R6.2, R7.1; no longer C17.2, C18.2, J2.1, J3.5, R6.1, R7.2
- net N$1: now also C4.1, R1.2; no longer C2.1, R2.2
- net N$10: now also C2.1; no longer C6.1
- net N$15: now also C14.1, C15.1; no longer C16.1, C17.1
- net N$8: now also R6.1; no longer R7.1
- net N$9: now also C1.1; no longer C5.1
- net OV: now also J1.5; no longer J2.5
- net SHD: now also J1.4; no longer J2.4
- net TCK: now also J2.4; no longer J3.4
- net TDO: now also J2.6; no longer J3.6
- net TMS: now also J2.2; no longer J3.2
- net TRIG: now also J1.3; no longer J2.3
- net VCAP: now also J1.6; no longer J2.6
- net VCC: now also C3.1, C5.1, C6.1, J1.2, J2.1, R2.2; no longer C1.1, C14.1, C15.1, J2.2, J3.1, R1.2
- net V_TIMER: now also C16.1, R7.2; no longer C18.1, R6.2
