File: hardware/gecko_power_supply/rev_e/monjolo.brd (EAGLE design)
At the start: 38.1 x 15.2 mm, 32 parts, among them Q2 DUAL_MOSFET_NP, Q3 DUAL_MOSFET_NP, U1 MN1382S 2.0V, U2 TC54VC 2.9V, U3 MCP1640T

Commit message: Updated monjolo solar rev e
Parts:
- moved U$1 0.51 mm to (8.00, 12.4)
Routing:
- net VCAP: track 48.5 -> 55.0 mm, vias 0 -> 1
- net GND: track 37.3 -> 41.5 mm
- net N$13: track 29.2 -> 28.2 mm
Changed lines of the file:
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@@
 <grid distance="0.05" unitdist="inch" unit="inch" style="lines" multiple="1" display="yes" altdistance="0.005" altunitdist="inch" altunit="inch"/>
 <layers>
-<layer number="1" name="Top" color="4" fill="1" visible="no" active="yes"/>
+<layer number="1" name="Top" color="4" fill="1" visible="yes" active="yes"/>
 <layer number="2" name="Route2" color="1" fill="3" visible="no" active="no"/>
 <layer number="3" name="Route3" color="4" fill="3" visible="no" active="no"/>
@@
 <layer number="14" name="Route14" color="1" fill="6" visible="no" active="no"/>
 <layer number="15" name="Route15" color="4" fill="6" visible="no" active="no"/>
-<layer number="16" name="Bottom" color="1" fill="1" visible="no" active="yes"/>
+<layer number="16" name="Bottom" color="1" fill="1" visible="yes" active="yes"/>
 <layer number="17" name="Pads" color="2" fill="1" visible="yes" active="yes"/>
 <layer number="18" name="Vias" color="2" fill="1" visible="yes" active="yes"/>
 <layer number="19" name="Unrouted" color="6" fill="1" visible="yes" active="yes"/>
 <layer number="20" name="Dimension" color="15" fill="1" visible="yes" active="yes"/>
-<layer number="21" name="tPlace" color="7" fill="1" visible="no" active="yes"/>
-<layer number="22" name="bPlace" color="7" fill="1" visible="no" active="yes"/>
-<layer number="23" name="tOrigins" color="15" fill="1" visible="no" active="yes"/>
-<layer number="24" name="bOrigins" color="15" fill="1" visible="no" active="yes"/>
-<layer number="25" name="tNames" color="7" fill="1" visible="no" active="yes"/>
-<layer number="26" name="bNames" color="7" fill="1" visible="no" active="yes"/>
+<layer number="21" name="tPlace" color="7" fill="1" visible="yes" active="yes"/>
+<layer number="22" name="bPlace" color="7" fill="1" visible="yes" active="yes"/>
+<layer number="23" name="tOrigins" color="15" fill="1" visible="yes" active="yes"/>
+<layer number="24" name="bOrigins" color="15" fill="1" visible="yes" active="yes"/>
+<layer number="25" name="tNames" color="7" fill="1" visible="yes" active="yes"/>
+<layer number="26" name="bNames" color="7" fill="1" visible="yes" active="yes"/>
 <layer number="27" name="tValues" color="7" fill="1" visible="no" active="yes"/>
 <layer number="28" name="bValues" color="7" fill="1" visible="no" active="yes"/>
@@
 <layer number="49" name="Reference" color="7" fill="1" visible="no" active="yes"/>
 <layer number="50" name="dxf" color="7" fill="1" visible="no" active="yes"/>
-<layer number="51" name="tDocu" color="14" fill="1" visible="no" active="yes"/>
-<layer number="52" name="bDocu" color="14" fill="1" visible="no" active="yes"/>
+<layer number="51" name="tDocu" color="14" fill="1" visible="yes" active="yes"/>
+<layer number="52" name="bDocu" color="14" fill="1" visible="yes" active="yes"/>
 <layer number="53" name="tGND_GNDA" color="7" fill="9" visible="no" active="no"/>
 <layer number="54" name="bGND_GNDA" color="1" fill="9" visible="no" active="no"/>
@@
 <wire x1="0" y1="15.24" x2="0" y2="0" width="0" layer="20"/>
 <wire x1="0" y1="0" x2="38.1" y2="0" width="0" layer="20"/>
-<text x="12.446" y="13.081" size="1.27" layer="21" font="vector" ratio="14">Solar Monjolo</text>
-<text x="24.892" y="0.889" size="1.016" layer="21" font="vector" ratio="12">LY, PKD, BC</text>
+<text x="11.684" y="13.081" size="1.27" layer="21" font="vector" ratio="14">Solar Monjolo</text>
+<text x="24.892" y="0.508" size="1.016" layer="21" font="vector" ratio="12">LY, PKD, BC</text>
 <text x="36.195" y="1.27" size="1.016" layer="21" font="vector" ratio="12">E</text>
 <text x="32.512" y="11.303" size="0.6096" layer="27">VCAP</text>
@@
 </element>
 <element name="D2" library="umich" package="LED-0603" value="" x="36.957" y="3.937" smashed="yes" rot="MR0">
-<attribute name="NAME" x="35.433" y="4.318" size="0.635" layer="26" font="vector" ratio="10" rot="MR0"/>
+<attribute name="NAME" x="36.068" y="4.572" size="0.635" layer="26" font="vector" ratio="10" rot="MR270"/>
 <attribute name="VALUE" x="35.687" y="2.667" size="1.016" layer="28" font="vector" ratio="12" rot="MR0"/>
 </element>
@@
 <attribute name="VALUE" x="14.986" y="4.567" size="0.6096" layer="27" font="vector" ratio="12"/>
 </element>
-<element name="U$1" library="logos" package="UMICH_SOLID_75MIL" value="UMICH_SOLID_SMALL" x="8.509" y="12.446"/>
+<element name="U$1" library="logos" package="UMICH_SOLID_75MIL" value="UMICH_SOLID_SMALL" x="8.001" y="12.446"/>
 <element name="C3" library="Gecko" package="CAP1210" value="100uF" x="2.794" y="10.795" smashed="yes" rot="R270">
 <attribute name="VALUE" value="" x="2.794" y="10.795" size="1.778" layer="27" rot="R270" display="off"/>
@@
 <contactref element="R10" pad="2"/>
 <contactref element="U3" pad="2"/>
-<wire x1="7.239" y1="11.2522" x2="7.239" y2="12.065" width="0.381" layer="1"/>
-<wire x1="6.6802" y1="10.541" x2="7.239" y2="11.2522" width="0.381" layer="1"/>
-<wire x1="7.239" y1="12.065" x2="7.239" y2="13.081" width="0.381" layer="1"/>
+<wire x1="6.223" y1="11.811" x2="7.366" y2="11.811" width="0.381" layer="1"/>
 <wire x1="20.447" y1="9.017" x2="21.463" y2="9.017" width="0.381" layer="1"/>
 <wire x1="21.463" y1="9.017" x2="21.59" y2="9.144" width="0.381" layer="1"/>
@@
 <wire x1="24.384" y1="3.175" x2="25.908" y2="3.175" width="0.381" layer="1"/>
 <wire x1="25.908" y1="3.175" x2="25.654" y2="3.302" width="0.381" layer="1"/>
-<via x="7.239" y="12.065" extent="1-16" drill="0.381"/>
+<via x="6.223" y="11.811" extent="1-16" drill="0.381"/>
 <via x="20.955" y="1.905" extent="1-16" drill="0.381"/>
 <via x="19.812" y="1.905" extent="1-16" drill="0.381"/>
 <via x="17.399" y="8.001" extent="1-16" drill="0.381"/>
 <via x="21.59" y="9.144" extent="1-16" drill="0.381"/>
-<via x="7.239" y="13.081" extent="1-16" drill="0.381"/>
+<via x="7.366" y="11.811" extent="1-16" drill="0.381"/>
 <via x="17.399" y="9.144" extent="1-16" drill="0.381"/>
 <via x="21.59" y="8.128" extent="1-16" drill="0.381"/>
@@
 <wire x1="16.383" y1="8.763" x2="12.827" y2="8.763" width="0.381" layer="1"/>
 <wire x1="12.827" y1="8.763" x2="12.573" y2="8.509" width="0.381" layer="1"/>
-<wire x1="19.812" y1="1.905" x2="17.145" y2="3.556" width="0" layer="19" extent="1-1"/>
+<wire x1="17.145" y1="3.556" x2="17.145" y2="2.286" width="0.4064" layer="1"/>
+<wire x1="17.145" y1="2.286" x2="17.78" y2="1.651" width="0.4064" layer="1"/>
+<wire x1="17.78" y1="1.651" x2="19.558" y2="1.651" width="0.4064" layer="1"/>
+<wire x1="19.558" y1="1.651" x2="19.812" y2="1.905" width="0.4064" layer="1"/>
+<wire x1="6.6802" y1="10.541" x2="6.6802" y2="11.3538" width="0.4064" layer="1"/>
+<wire x1="6.6802" y1="11.3538" x2="6.223" y2="11.811" width="0.4064" layer="1"/>
 </signal>
 <signal name="N$9">
@@
 <wire x1="28.702" y1="11.049" x2="32.004" y2="14.351" width="0.381" layer="1"/>
 <wire x1="32.004" y1="14.351" x2="33.02" y2="14.351" width="0.381" layer="1"/>
-<wire x1="4.344" y1="2.032" x2="2.56" y2="1.758" width="0" layer="19" extent="1-16"/>
+<wire x1="2.56" y1="1.758" x2="4.231" y2="3.429" width="0.8128" layer="16"/>
+<wire x1="4.231" y1="3.429" x2="6.096" y2="3.429" width="0.8128" layer="16"/>
+<via x="6.096" y="3.429" extent="1-16" drill="0.508"/>
+<wire x1="6.096" y1="3.429" x2="5.741" y2="3.429" width="0.8128" layer="1"/>
+<wire x1="5.741" y1="3.429" x2="4.344" y2="2.032" width="0.8128" layer="1"/>
 </signal>
 <signal name="N$12">
@@
 <wire x1="11.8364" y1="10.16" x2="10.795" y2="9.1186" width="0.381" layer="1"/>
 <wire x1="10.795" y1="9.1186" x2="10.795" y2="8.509" width="0.381" layer="1"/>
-<wire x1="14.986" y1="11.176" x2="14.986" y2="12.192" width="0.381" layer="16"/>
-<wire x1="14.986" y1="12.192" x2="15.875" y2="13.081" width="0.381" layer="16"/>
-<wire x1="15.875" y1="13.081" x2="35.433" y2="13.081" width="0.381" layer="16"/>
-<wire x1="35.433" y1="13.081" x2="35.941" y2="12.573" width="0.381" layer="16"/>
-<wire x1="35.941" y1="12.573" x2="36.957" y2="12.573" width="0.381" layer="16"/>
+<wire x1="36.957" y1="12.573" x2="16.383" y2="12.573" width="0.381" layer="16"/>
+<wire x1="16.383" y1="12.573" x2="14.986" y2="11.176" width="0.381" layer="16"/>
 </signal>
 <signal name="N$14">
