File: hardware/impulse/rev_a/impulse.brd (EAGLE design)
At the start: 32.5 x 13 mm, 45 parts, among them J1 GECKO_POWER_SUPPLY_CONN, J3 EPIC-PROG-POGO-NO-LEGS, Q1 MOSFET-NCHANNELXFDN-3, U1 DS2411, U2 FM25LBTDFN-8, U4 MSP430F1611IRTD, U5 CC2420RGZ, X1 TXC-7V

Commit message: getting closer
all the parts are on the board
Parts:
- moved R4 19.9 mm to (26.6, 5.41), flipped to the bottom, turned to 270 degrees
- moved C5 19.8 mm to (25.6, 5.44), flipped to the bottom, turned to 270 degrees
- moved R7 13.4 mm to (25.7, 11.9), turned to 270 degrees
- moved Q1 13.0 mm to (23.4, 12.0)
- moved C16 12.8 mm to (24.8, 11.9), turned to 90 degrees
- moved U2 12.5 mm to (27.0, 9.11), flipped to the bottom, turned to 180 degrees
- moved R8 12.3 mm to (22.1, 11.9), turned to 270 degrees
- moved C1 12.1 mm to (27.6, 9.80), turned to 0 degrees
- moved R6 12.0 mm to (15.1, 8.79), turned to 90 degrees
- moved C2 11.8 mm to (27.6, 10.7), turned to 0 degrees
- moved R9 9.43 mm to (20.7, 0.51)
- moved U1 9.33 mm to (20.5, 10.8), flipped to the bottom, turned to 90 degrees
- moved R2 9.17 mm to (22.7, 10.8), flipped to the bottom, turned to 270 degrees
- moved C3 8.64 mm to (28.4, 8.03), turned to 90 degrees
- moved R3 6.52 mm to (26.0, 12.4), flipped to the bottom, turned to 180 degrees
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Connections:
- removed net DS2411: R2.1, U1.1
- net ONEWIRE: now also R2.1, U1.1
- net TIME_CTL: now also R8.2, U4.4, U4.5
- net V_TIMER: no longer R8.2
Routing:
- net RADIO_VREG_EN: track 2.91 -> 25.6 mm, vias 0 -> 2
- net UART1TX: track 0.00 -> 20.7 mm, vias 0 -> 3
- net UART1RX: track 0.00 -> 18.2 mm, vias 0 -> 2
- net !RADIO_CS: track 1.40 -> 14.3 mm, vias 0 -> 2
- net !RESET: track 0.00 -> 9.56 mm
- net TCK: track 0.00 -> 6.99 mm, vias 0 -> 2
- net N$1: track 0.00 -> 4.10 mm
- net VCC: track 3.03 -> 6.40 mm
- net TIME_CTL: track 0.00 -> 2.19 mm
- net V_TIMER: track 0.00 -> 2.18 mm
- net RADIO_CCA: track 11.0 -> 9.57 mm
- net RADIO_FIFOP: track 12.2 -> 10.8 mm
- net N$8: track 28.5 -> 29.6 mm
- net RADIO_FIFO: track 11.3 -> 10.6 mm
- net SCLK0: track 8.67 -> 9.31 mm, vias 2 -> 0
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
Commit message: routed
Parts:
- moved C8 1.81 mm to (13.2, 3.91), turned to 0 degrees
- moved C4 1.35 mm to (13.2, 3.05), turned to 0 degrees
- moved C5 0.18 mm to (25.4, 5.44)
Routing:
- net !FRAM_WP: track 0.00 -> 26.1 mm, vias 0 -> 1
- net MOSI0: track 8.46 -> 24.3 mm, vias 0 -> 1
- net SCLK0: track 9.31 -> 25.0 mm, vias 0 -> 1
- net MISO0: track 9.28 -> 23.9 mm
- net !FRAM_CS: track 0.00 -> 13.9 mm, vias 0 -> 1
- net ONEWIRE: track 0.00 -> 9.56 mm, vias 0 -> 1
- net UART1TX: track 20.7 -> 11.9 mm
- net !FRAM_HOLD: track 0.00 -> 5.43 mm, vias 0 -> 1
- net VCC: track 6.40 -> 9.13 mm
- net N$8: track 29.6 -> 28.4 mm
- net !RADIO_CS: track 14.3 -> 15.2 mm
- net RADIO_SFD: track 10.3 -> 11.0 mm
- net TCK: track 6.99 -> 6.35 mm, vias 2 -> 0
- net RADIO_VREG_EN: track 25.6 -> 26.2 mm

Commit message: pwr and gnd routed
Parts:
- moved R11 13.7 mm to (23.0, 0.61), turned to 0 degrees
- moved R10 10.9 mm to (12.0, 1.17), turned to 0 degrees
- moved R6 1.26 mm to (16.1, 7.92)
- moved R8 0.69 mm to (21.4, 11.9)
- moved C4 0.61 mm to (13.8, 3.05)
- moved C8 0.61 mm to (13.8, 3.91)
- moved R5 0.51 mm to (28.4, 12.4), turned to 0 degrees
- moved R13 0.41 mm to (9.93, 12.0)
- moved R9 0.28 mm to (20.4, 0.58)
- moved C14 0.28 mm to (13.6, 8.99)
- moved C9 0.28 mm to (13.6, 8.26)
- moved R1 0.23 mm to (27.4, 7.80)
- moved C3 0.23 mm to (28.4, 7.80)
- moved C12 0.20 mm to (3.30, 9.42)
- moved C5 0.15 mm to (25.6, 5.44)
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Connections:
- net TIME_CTL: no longer U4.4, U4.48
- net V_TIMER: now also U4.61; no longer U4.59
Routing:
- net N$8: track 28.4 -> 54.3 mm, vias 0 -> 3
- net VCC: track 9.13 -> 26.7 mm, vias 0 -> 9
- net !RADIO_RESET: track 1.22 -> 17.1 mm, vias 0 -> 2
- net GND: track 11.7 -> 21.6 mm, vias 0 -> 71
- net UART1TX: track 11.9 -> 21.1 mm
- net V_TIMER: track 2.18 -> 10.5 mm, vias 0 -> 2
- net RADIO_VREG_EN: track 26.2 -> 24.3 mm, vias 2 -> 4
- net N$1: track 3.64 -> 2.40 mm
- net !FRAM_CS: track 13.9 -> 12.9 mm
- net UART1RX: track 18.3 -> 19.0 mm
- net !FRAM_WP: track 26.1 -> 26.8 mm
- net !RADIO_CS: track 15.2 -> 14.5 mm
- net TIME_CTL: track 2.19 -> 2.79 mm

Commit message: routed. silkscreen. wow.
Parts:
- removed C21: 22pF, passives:0402_CAP
- removed U5: CC2420RGZ, chips:S-PVQFN-N48
- added C19: 2.2uF, passives:0402_CAP
- added D1: (no value), SparkFun-LED:LED-0603
- added R14: 4.7M, passives:0402_RES
- added U3: MSP430F1611IRTD, chips:S-PVQFN-N64
- C1: value 0.1uF -> 12pF
- C10, C14, C15, C18: value 68pF -> 0.1uF
- C13: value 0.01uF -> 0.1uF
- C16: value 2.2uF -> 0.1uF
- C17: value 12pF -> 0.1uF
- C2, C3: value 0.1uF -> 22pF
- C20: value 22pF -> 10uF; device passives:0402_CAP -> rcl:C0805
- C4, C5, C6: value 0.1uF -> 68pF
- C7: value (none) -> 68pF; device rcl:C0805 -> passives:0402_CAP
- C8: value 0.1uF -> 0.01uF
- R1: value 100k -> 2.2
- R12: value 43k -> 1M
- R13: value 2.2 -> 1M
- R2: value 2.2k -> 470
- R3: value 4.7k -> 2.2k
- R6: value 100k -> 4.7k
- R7: value 4.7M -> 43k
- R8, R9: value 1M -> 100k
- U4: value MSP430F1611IRTD -> CC2420RGZ; device chips:S-PVQFN-N64 -> chips:S-PVQFN-N48
- moved U$1 32.9 mm to (32.3, 1.45), turned to 90 degrees
- moved C1 26.2 mm to (1.55, 7.29), turned to 90 degrees
- moved C13 23.7 mm to (27.6, 10.5), turned to 0 degrees
- moved C18 21.2 mm to (25.6, 5.44), flipped to the bottom, turned to 270 degrees
- moved C10 21.1 mm to (27.6, 9.65), turned to 0 degrees
- moved R12 20.3 mm to (26.6, 11.7), turned to 90 degrees
- moved R7 19.4 mm to (6.30, 11.5)
- moved R1 17.9 mm to (9.93, 12.0), turned to 90 degrees
- moved C16 16.4 mm to (8.38, 11.5)
- moved C2 15.8 mm to (11.9, 12.0), turned to 90 degrees
- moved R13 15.5 mm to (20.4, 0.58), turned to 180 degrees
- moved C14 14.8 mm to (28.3, 7.75), turned to 90 degrees
- moved U4 13.4 mm to (8.05, 6.20), turned to 0 degrees
- moved R6 13.3 mm to (28.5, 12.4), flipped to the bottom, turned to 180 degrees
- moved C17 12.7 mm to (13.8, 3.91), turned to 0 degrees
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- renumbered A2 to A1, J3 to J2, L2 to L1
Connections:
- new net N$6: D1.A, R2.1
- new net N$9: R2.2, U3.60
- net !FRAM_CS: now also R6.1, U3.44; no longer R3.1, U4.44
- net !FRAM_HOLD: now also U3.51; no longer U4.51
- net !FRAM_WP: now also U3.32; no longer U4.32
- net !RADIO_CS: now also R13.2, U3.38, U4.31; no longer R9.2, U4.38, U5.31
- net !RADIO_RESET: now also U3.42, U4.21; no longer U4.42, U5.21
- net !RESET: now also C14.1, R9.2, U3.58; no longer C3.1, R1.2, U4.58
- net GND: now also C19.2, D1.C, R14.1, U3.62, U3.63, U3.GND, U4.19, U4.22, U4.23, U4.24, U4.5, U4.9, U4.VSS_QFN; no longer C21.2, R8.1, U4.62, U4.63, U4.GND, U5.19, U5.22, U5.23, U5.24, U5.5, U5.9, U5.VSS_QFN
- net MISO0: now also U3.30, U4.34; no longer U4.30, U5.34
- net MOSI0: now also U3.29, U4.33; no longer U4.29, U5.33
- net N$1: now also R8.1, U3.25; no longer R6.1, U4.25
- net N$12: now also C1.1, U4.7; no longer C17.1, U5.7
- net N$17: now also U4.8; no longer U5.8
- net N$18: now also U4.6; no longer U5.6
- net N$19: now also C3.1, U4.38; no longer C21.1, U5.38
- net N$20: now also C2.1, U4.39; no longer C20.1, U5.39
- net N$5: now also R7.2, U4.45; no longer R12.2, U5.45
- net N$7: now also C20.1, R1.2; no longer C7.1, R13.2
- net N$8: now also C17.1, C4.1, C5.1, C6.1, C7.1, R1.1, U4.1, U4.10, U4.14, U4.15, U4.17, U4.18, U4.2, U4.20, U4.26, U4.3, U4.35, U4.37, U4.4, U4.42, U4.44, U4.48; no longer C10.1, C13.1, C14.1, C15.1, C18.1, R13.1, U5.1, U5.10, U5.14, U5.15, U5.17, U5.18, U5.2, U5.20, U5.26, U5.3, U5.35, U5.37, U5.4, U5.42, U5.44, U5.48
- net ONEWIRE: now also R3.1, U3.24; no longer R2.1, U4.24
- net RADIO_CCA: now also U3.16, U4.28; no longer U4.16, U5.28
- net RADIO_FIFO: now also U3.15, U4.30; no longer U4.15, U5.30
- net RADIO_FIFOP: now also U3.12, U4.29; no longer U4.12, U5.29
- net RADIO_SFD: now also U3.37, U4.27; no longer U4.37, U5.27
- net RADIO_VREG_EN: now also U3.41; no longer U5.41
- net SCLK0: now also U3.31, U4.32; no longer U4.31, U5.32
- net TCK: now also U3.57; no longer U4.57
- net TIME_CTL: now also R12.2, U3.5; no longer R8.2, U4.5
- net UART1RX: now also U3.22, U3.35; no longer U4.22, U4.35
- net UART1TX: now also U3.13, U3.34; no longer U4.13, U4.34
- net VCC: now also C10.1, C13.1, C15.1, C16.1, C18.1, R13.1, R8.2, U3.1, U3.64, U4.25, U4.43; no longer C1.1, C2.1, C4.1, C5.1, C6.1, R1.1, R2.2, U4.1, U4.64, U5.25, U5.43
- net V_TIMER: now also C19.1, R14.2, U3.61; no longer C16.1, R7.2, U4.61
Routing:
- net GND: track 21.6 -> 31.9 mm
- net N$9: track 0.00 -> 3.91 mm
- net TIME_CTL: track 2.79 -> 6.07 mm
- net !FRAM_CS: track 12.9 -> 15.9 mm
- net V_TIMER: track 10.5 -> 7.84 mm, vias 2 -> 0
- net !RESET: track 9.48 -> 10.5 mm
- net N$6: track 0.00 -> 1.02 mm
- net !FRAM_WP: track 26.8 -> 27.5 mm
- net MOSI0: track 24.3 -> 23.7 mm
- net VCC: track 26.7 -> 26.9 mm, vias 9 -> 10
Other:
- board text added: "2013/09/19"
- board text added: "A"
- board text added: "Activator"
- board text removed: "2013/08/14"
