File: hardware/impulse/rev_a/impulse.sch (EAGLE design)
At the start: 45 parts, among them J1 GECKO_POWER_SUPPLY_CONN, J3 EPIC-PROG-POGO-NO-LEGS, Q1 MOSFET-NCHANNELXFDN-3, U1 DS2411, U2 FM25LBTDFN-8, U4 MSP430F1611IRTD, U5 CC2420RGZ, X1 TXC-7V

Commit message: getting closer
all the parts are on the board
Connections:
- removed net DS2411: R2.1, U1.I/O
- net ONEWIRE: now also R2.1, U1.I/O
- net TIME_CTL: now also R8.2, U4.P6.5/A5, U4.P6.6/A6/DAC0
- net V_TIMER: no longer R8.2
Other:
- moved on the sheet: R8
Changed lines of the file:
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@@
 <instance part="P+13" gate="VCC" x="274.32" y="137.16"/>
 <instance part="GND10" gate="1" x="309.88" y="121.92"/>
-<instance part="R8" gate="G$1" x="266.7" y="215.9" rot="R90"/>
-<instance part="GND31" gate="1" x="266.7" y="205.74"/>
+<instance part="R8" gate="G$1" x="261.62" y="215.9" rot="R90"/>
+<instance part="GND31" gate="1" x="261.62" y="205.74"/>
 <instance part="C17" gate="G$1" x="233.68" y="48.26" smashed="yes">
 <attribute name="NAME" x="237.998" y="39.878" size="1.778" layer="95" ratio="12" rot="R90" align="bottom-center"/>
@@
 <pinref part="R8" gate="G$1" pin="1"/>
 <pinref part="GND31" gate="1" pin="GND"/>
-<wire x1="266.7" y1="210.82" x2="266.7" y2="208.28" width="0.1524" layer="91"/>
+<wire x1="261.62" y1="210.82" x2="261.62" y2="208.28" width="0.1524" layer="91"/>
 </segment>
 </net>
@@
 </segment>
 </net>
-<net name="DS2411" class="0">
-<segment>
-<pinref part="U1" gate="G$1" pin="I/O"/>
-<wire x1="304.8" y1="88.9" x2="317.5" y2="88.9" width="0.1524" layer="91"/>
-<label x="322.58" y="88.9" size="1.27" layer="95" xref="yes"/>
-<pinref part="R2" gate="G$1" pin="1"/>
-<wire x1="317.5" y1="88.9" x2="322.58" y2="88.9" width="0.1524" layer="91"/>
-<wire x1="317.5" y1="91.44" x2="317.5" y2="88.9" width="0.1524" layer="91"/>
-<junction x="317.5" y="88.9"/>
-</segment>
-</net>
 <net name="V_TIMER" class="0">
 <segment>
@@
 <junction x="281.94" y="226.06"/>
 <pinref part="Q1" gate="G$1" pin="S"/>
-<wire x1="276.86" y1="226.06" x2="266.7" y2="226.06" width="0.1524" layer="91"/>
+<wire x1="276.86" y1="226.06" x2="274.32" y2="226.06" width="0.1524" layer="91"/>
 <junction x="276.86" y="226.06"/>
-<label x="259.08" y="226.06" size="1.27" layer="95" rot="R180" xref="yes"/>
-<pinref part="R8" gate="G$1" pin="2"/>
-<wire x1="266.7" y1="226.06" x2="259.08" y2="226.06" width="0.1524" layer="91"/>
-<wire x1="266.7" y1="220.98" x2="266.7" y2="226.06" width="0.1524" layer="91"/>
-<junction x="266.7" y="226.06"/>
+<label x="274.32" y="226.06" size="1.27" layer="95" rot="R180" xref="yes"/>
 </segment>
 <segment>
@@
 <segment>
 <pinref part="Q1" gate="G$1" pin="G"/>
-<wire x1="274.32" y1="233.68" x2="271.78" y2="233.68" width="0.1524" layer="91"/>
-<label x="271.78" y="233.68" size="1.27" layer="95" rot="R180" xref="yes"/>
+<wire x1="274.32" y1="233.68" x2="261.62" y2="233.68" width="0.1524" layer="91"/>
+<label x="259.08" y="233.68" size="1.27" layer="95" rot="R180" xref="yes"/>
+<pinref part="R8" gate="G$1" pin="2"/>
+<wire x1="261.62" y1="233.68" x2="259.08" y2="233.68" width="0.1524" layer="91"/>
+<wire x1="261.62" y1="220.98" x2="261.62" y2="233.68" width="0.1524" layer="91"/>
+<junction x="261.62" y="233.68"/>
 </segment>
 <segment>
@@
 <wire x1="86.36" y1="78.74" x2="88.9" y2="78.74" width="0.1524" layer="91"/>
 <label x="88.9" y="78.74" size="1.27" layer="95" xref="yes"/>
+</segment>
+<segment>
+<pinref part="U4" gate="G$1" pin="P6.5/A5"/>
+<wire x1="86.36" y1="53.34" x2="88.9" y2="53.34" width="0.1524" layer="91"/>
+<label x="88.9" y="53.34" size="1.27" layer="95" xref="yes"/>
+</segment>
+<segment>
+<pinref part="U4" gate="G$1" pin="P6.6/A6/DAC0"/>
+<wire x1="86.36" y1="50.8" x2="88.9" y2="50.8" width="0.1524" layer="91"/>
+<label x="88.9" y="50.8" size="1.27" layer="95" xref="yes"/>
 </segment>
 </net>
@@
 <label x="20.32" y="78.74" size="1.27" layer="95" rot="MR0" xref="yes"/>
 </segment>
-</net>
+<segment>
+<pinref part="U1" gate="G$1" pin="I/O"/>
+<wire x1="304.8" y1="88.9" x2="317.5" y2="88.9" width="0.1524" layer="91"/>
+<label x="322.58" y="88.9" size="1.27" layer="95" xref="yes"/>
+<pinref part="R2" gate="G$1" pin="1"/>
+<wire x1="317.5" y1="88.9" x2="322.58" y2="88.9" width="0.1524" layer="91"/>
+<wire x1="317.5" y1="91.44" x2="317.5" y2="88.9" width="0.1524" layer="91"/>
+<junction x="317.5" y="88.9"/>
+</segment>
+</net>

Commit message: pwr and gnd routed
Connections:
- net TIME_CTL: no longer U4.P5.4/MCLK, U4.P6.5/A5
- net V_TIMER: now also U4.P6.2/A2; no longer U4.P6.0/A0
Changed lines of the file:
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@@
 </segment>
 <segment>
-<pinref part="U4" gate="G$1" pin="P6.0/A0"/>
-<wire x1="86.36" y1="66.04" x2="88.9" y2="66.04" width="0.1524" layer="91"/>
-<label x="88.9" y="66.04" size="1.27" layer="95" xref="yes"/>
+<pinref part="U4" gate="G$1" pin="P6.2/A2"/>
+<wire x1="86.36" y1="60.96" x2="88.9" y2="60.96" width="0.1524" layer="91"/>
+<label x="88.9" y="60.96" size="1.27" layer="95" xref="yes"/>
 </segment>
 </net>
@@
 </segment>
 <segment>
-<pinref part="U4" gate="G$1" pin="P5.4/MCLK"/>
-<wire x1="86.36" y1="78.74" x2="88.9" y2="78.74" width="0.1524" layer="91"/>
-<label x="88.9" y="78.74" size="1.27" layer="95" xref="yes"/>
-</segment>
-<segment>
-<pinref part="U4" gate="G$1" pin="P6.5/A5"/>
-<wire x1="86.36" y1="53.34" x2="88.9" y2="53.34" width="0.1524" layer="91"/>
-<label x="88.9" y="53.34" size="1.27" layer="95" xref="yes"/>
-</segment>
-<segment>

Commit message: routed. silkscreen. wow.
Parts:
- removed C21: 22pF, passives:CAPACITOR
- removed J3: EPIC-PROG-POGO-NO-LEGS, epic:EPIC-PROG-POGO-NO-LEGS
- removed U5: CC2420RGZ, chips:CC2420RGZ
- added C19: 2.2uF, passives:CAPACITOR
- added D1: (no value), SparkFun-LED:LED0603
- added J2: EPIC-PROG-POGO-NO-LEGS, epic:EPIC-PROG-POGO-NO-LEGS
- added R14: 4.7M, passives:RESISTOR
- added U3: MSP430F1611IRTD, chips:MSP430F1611IRTD
- C1: value 0.1uF -> 12pF
- C10, C14, C15, C18: value 68pF -> 0.1uF
- C13: value 0.01uF -> 0.1uF
- C16: value 2.2uF -> 0.1uF
- C17: value 12pF -> 0.1uF
- C2, C3: value 0.1uF -> 22pF
- C20: value 22pF -> 10uF; device passives:CAPACITOR -> rcl:C-USC0805; DIGIKEY (none) -> 478-2561-1-ND
- C4, C5, C6: value 0.1uF -> 68pF
- C7: value (none) -> 68pF; device rcl:C-USC0805 -> passives:CAPACITOR; DIGIKEY 478-2561-1-ND -> (none)
- C8: value 0.1uF -> 0.01uF
- R1: value 100k -> 2.2
- R12: value 43k -> 1M
- R13: value 2.2 -> 1M
- R2: value 2.2k -> 470
- R3: value 4.7k -> 2.2k
- R6: value 100k -> 4.7k
- R7: value 4.7M -> 43k
- R8, R9: value 1M -> 100k
- U4: value MSP430F1611IRTD -> CC2420RGZ; device chips:MSP430F1611IRTD -> chips:CC2420RGZ
- renumbered A2 to A1, L2 to L1
Connections:
- new net N$6: D1.A, R2.1
- new net N$9: R2.2, U3.P6.1/A1
- net !FRAM_CS: now also R6.1, U3.P5.0/STE1; no longer R3.1, U4.P5.0/STE1
- net !FRAM_HOLD: now also U3.P5.7/TBOUTH/SVSOUT; no longer U4.P5.7/TBOUTH/SVSOUT
- net !FRAM_WP: now also U3.P3.4/UTXD0; no longer U4.P3.4/UTXD0
- net !RADIO_CS: now also R13.2, U3.P4.2/TB2, U4.CSN; no longer R9.2, U4.P4.2/TB2, U5.CSN
- net !RADIO_RESET: now also U3.P4.6/TB6, U4.RESETN; no longer U4.P4.6/TB6, U5.RESETN
- net !RESET: now also C14.1, J2.RST#, R9.2, U3.RST/NMI; no longer C3.1, J3.RST#, R1.2, U4.RST/NMI
- net GND: now also C19.2, D1.C, J2.GND, R14.1, U3.AVSS, U3.DVSS1, U4.AGND, U4.DGND, U4.DGND_GUARD, U4.DSUB_CORE, U4.DSUB_PADS, U4.GND, U4.GND2; no longer C21.2, J3.GND, R8.1, U4.AVSS, U4.DVSS1, U5.AGND, U5.DGND, U5.DGND_GUARD, U5.DSUB_CORE, U5.DSUB_PADS, U5.GND, U5.GND2
- net MISO0: now also U3.P3.2/MISO0, U4.SO; no longer U4.P3.2/MISO0, U5.SO
- net MOSI0: now also U3.P3.1/MOSI0/SDA, U4.SI; no longer U4.P3.1/MOSI0/SDA, U5.SI
- net N$1: now also R8.1, U3.P2.5/ROSC; no longer R6.1, U4.P2.5/ROSC
- net N$12: now also C1.1, U4.TXRX_SWITCH; no longer C17.1, U5.TXRX_SWITCH
- net N$17: now also U4.RF_N; no longer U5.RF_N
- net N$18: now also U4.RF_P; no longer U5.RF_P
- net N$19: now also C3.1, U4.XOSC16_Q2; no longer C21.1, U5.XOSC16_Q2
- net N$20: now also C2.1, U4.XOSC16_Q1; no longer C20.1, U5.XOSC16_Q1
- net N$5: now also R7.2, U4.R_BIAS; no longer R12.2, U5.R_BIAS
- net N$7: now also C20.1, R1.2; no longer C7.1, R13.2
- net N$8: now also C17.1, C4.1, C5.1, C6.1, C7.1, R1.1, U4.AVDD_ADC, U4.AVDD_CHP, U4.AVDD_IF1, U4.AVDD_IF2, U4.AVDD_PRE, U4.AVDD_RF1, U4.AVDD_RF2, U4.AVDD_SW, U4.AVDD_VCO, U4.AVDD_XOSC16, U4.DGUARD, U4.DVDD1.8, U4.DVDD_ADC, U4.DVDD_RAM, U4.VCO_GUARD, U4.VREG_OUT; no longer C10.1, C13.1, C14.1, C15.1, C18.1, R13.1, U5.AVDD_ADC, U5.AVDD_CHP, U5.AVDD_IF1, U5.AVDD_IF2, U5.AVDD_PRE, U5.AVDD_RF1, U5.AVDD_RF2, U5.AVDD_SW, U5.AVDD_VCO, U5.AVDD_XOSC16, U5.DGUARD, U5.DVDD1.8, U5.DVDD_ADC, U5.DVDD_RAM, U5.VCO_GUARD, U5.VREG_OUT
- net ONEWIRE: now also R3.1, U3.P2.4/CA1/TA2; no longer R2.1, U4.P2.4/CA1/TA2
- net RADIO_CCA: now also U3.P1.4/SMCLK, U4.CCA; no longer U4.P1.4/SMCLK, U5.CCA
- net RADIO_FIFO: now also U3.P1.3/TA2, U4.FIFO; no longer U4.P1.3/TA2, U5.FIFO
- net RADIO_FIFOP: now also U3.P1.0/TACLK, U4.FIFOP; no longer U4.P1.0/TACLK, U5.FIFOP
- net RADIO_SFD: now also U3.P4.1/TB1, U4.SFD; no longer U4.P4.1/TB1, U5.SFD
- net RADIO_VREG_EN: now also U3.P4.5/TB5, U4.VREG_EN; no longer U4.P4.5/TB5, U5.VREG_EN
- net SCLK0: now also U3.P3.3/UCLK0/SCL, U4.SCLK; no longer U4.P3.3/UCLK0/SCL, U5.SCLK
- net TCK: now also J2.TCK, U3.TCK; no longer J3.TCK, U4.TCK
- net TIME_CTL: now also R12.2, U3.P6.6/A6/DAC0; no longer R8.2, U4.P6.6/A6/DAC0
- net UART1RX: now also J2.RX1, U3.P2.2/CAOUT/TA0/BSLRX, U3.P3.7/URXD1; no longer J3.RX1, U4.P2.2/CAOUT/TA0/BSLRX, U4.P3.7/URXD1
- net UART1TX: now also J2.TX1, U3.P1.1/TA0/BSLTX, U3.P3.6/UTXD1; no longer J3.TX1, U4.P1.1/TA0/BSLTX, U4.P3.6/UTXD1
- net VCC: now also C10.1, C13.1, C15.1, C16.1, C18.1, J2.VDD, R13.1, R8.2, U3.AVCC, U3.DVCC, U4.DVDD3.3, U4.VREG_IN; no longer C1.1, C2.1, C4.1, C5.1, C6.1, J3.VDD, R1.1, R2.2, U4.AVCC, U4.DVCC, U5.DVDD3.3, U5.VREG_IN
- net V_TIMER: now also C19.1, R14.2, U3.P6.2/A2; no longer C16.1, R7.2, U4.P6.2/A2
