File: hardware/impulse/rev_c/impulse.sch (EAGLE design)
At the start: 52 parts, among them J2 EPIC-PROG-POGO-NO-LEGS, J3 IMPULSE_GECKO_HEADER, Q1 MOSFET-NCHANNELXFDN-3, U1 DS2411, U2 FM25LBTDFN-8, U3 MSP430F1611IRTD, U4 CC2420RGZ, X1 TXC-7V, X2 ABRACON-ABS05

Commit message: updated rev c.
new solder jumpers

straightened some traces

added some vias for planes
Parts:
- removed R17: 0, passives:RESISTOR
- added SJ1, SJ2, SJ3: SJ, passives:SJ
Connections:
- new net N$10: J3.TRIGGER/P2.1, SJ1.P$1
- new net N$11: J3.SHTDWN/P2.0, SJ2.P$1
- net N$6: now also R2.2; no longer R2.1
- net OV: now also SJ3.P$2; no longer R17.2
- net OV-HEADER: now also SJ3.P$1; no longer R17.1
- net SHD: now also SJ2.P$2; no longer J3.SHTDWN/P2.0
- net TRIG: now also SJ1.P$2; no longer J3.TRIGGER/P2.1
- net VCC: now also R2.1; no longer R2.2
Other:
- note added: "DS2411 ID Chip"
- note added: "FRAM"
- note added: "Programming Connection"
- note added: "Timing Circuit"
- moved on the sheet: C18, C19, D1, D2, J2, Q1, R12, R14, R16, R2, R4, R5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
